Commit message: add packages in urdf

File: robot_simplified.urdf (robot description, URDF)
Before this commit: robot robot_v1, 24 links, 23 joints
Links:
- link urdf_base: geometry collision mesh filename=package://assets/b_base.stl; collision mesh filename=package://assets/f_base.stl
- link urdf_hip_assembly: geometry collision mesh filename=package://assets/hip.stl; visual mesh filename=package://assets/hip.stl
- link urdf_hip_assembly_2: geometry collision mesh filename=package://assets/hip.stl; visual mesh filename=package://assets/hip.stl
- link urdf_l_elbow_assembly: geometry collision mesh filename=package://assets/l_elbow.stl; visual mesh filename=package://assets/l_elbow.stl
- link urdf_l_lower_forearm_assembly: geometry collision mesh filename=package://assets/l_lower_forearm.stl; visual mesh filename=package://assets/l_lower_forearm.stl
- link urdf_l_shoulder_assembly: geometry collision mesh filename=package://assets/l_shoulder.stl; visual mesh filename=package://assets/l_shoulder.stl
- link urdf_l_tibia_assembly: geometry collision mesh filename=package://assets/foot.stl; collision mesh filename=package://assets/l_tibia.stl
- link urdf_l_upper_arm_assembly: geometry collision mesh filename=package://assets/l_upper_arm.stl; visual mesh filename=package://assets/l_upper_arm.stl
- link urdf_l_upper_femur_assembly: geometry collision mesh filename=package://assets/l_upper_femur.stl; visual mesh filename=package://assets/l_upper_femur.stl
- link urdf_l_upper_forearm_assembly: geometry collision mesh filename=package://assets/l_upper_forearm.stl; visual mesh filename=package://assets/l_upper_forearm.stl
- link urdf_l_wrist_assembly: geometry collision mesh filename=package://assets/l_hand.stl; collision mesh filename=package://assets/l_wrist.stl
- link urdf_lower_femur_assembly: geometry collision mesh filename=package://assets/lower_femur.stl; visual mesh filename=package://assets/lower_femur.stl
- link urdf_lower_femur_assembly_2: geometry collision mesh filename=package://assets/lower_femur.stl; visual mesh filename=package://assets/lower_femur.stl
- link urdf_r_elbow_assembly: geometry collision mesh filename=package://assets/r_elbow.stl; visual mesh filename=package://assets/r_elbow.stl
- link urdf_r_lower_forearm_assembly: geometry collision mesh filename=package://assets/r_lower_forearm.stl; visual mesh filename=package://assets/r_lower_forearm.stl
- link urdf_r_shoulder_assembly: geometry collision mesh filename=package://assets/r_shoulder.stl; visual mesh filename=package://assets/r_shoulder.stl
- link urdf_r_tibia_assembly: geometry collision mesh filename=package://assets/foot.stl; collision mesh filename=package://assets/r_tibia.stl
- link urdf_r_upper_arm_assembly: geometry collision mesh filename=package://assets/r_upper_arm.stl; visual mesh filename=package://assets/r_upper_arm.stl
- link urdf_r_upper_femur_assemby: geometry collision mesh filename=package://assets/r_upper_femur.stl; visual mesh filename=package://assets/r_upper_femur.stl
- link urdf_r_upper_forearm_assembly: geometry collision mesh filename=package://assets/r_upper_forearm.stl; visual mesh filename=package://assets/r_upper_forearm.stl
- link urdf_r_wrist_assembly: geometry collision mesh filename=package://assets/r_hand.stl; collision mesh filename=package://assets/r_wrist.stl
- link urdf_simplified_torso_sub_assembly: geometry collision mesh filename=package://assets/head.stl; collision mesh filename=package://assets/simplified_torso.stl
Joints:
- joint left_shoulder_roll_joint_X6: limit lower=-0.05533 upper=3.39626 effort=10 velocity=10 -> lower=-1.74533 upper=1.39626 effort=10 velocity=10

File: robot_with_limits.urdf (robot description, URDF)
Before this commit: robot robot_v1, 24 links, 23 joints
Links:
- link urdf_base: geometry collision mesh filename=package://assets/b_base.stl; collision mesh filename=package://assets/f_base.stl
- link urdf_hip_assembly: geometry collision mesh filename=package://assets/hip.stl; visual mesh filename=package://assets/hip.stl
- link urdf_hip_assembly_2: geometry collision mesh filename=package://assets/hip.stl; visual mesh filename=package://assets/hip.stl
- link urdf_l_elbow_assembly: geometry collision mesh filename=package://assets/l_elbow.stl; visual mesh filename=package://assets/l_elbow.stl
- link urdf_l_lower_forearm_assembly: geometry collision mesh filename=package://assets/l_lower_forearm.stl; visual mesh filename=package://assets/l_lower_forearm.stl
- link urdf_l_shoulder_assembly: geometry collision mesh filename=package://assets/l_shoulder.stl; visual mesh filename=package://assets/l_shoulder.stl
- link urdf_l_tibia_assembly: geometry collision mesh filename=package://assets/foot.stl; collision mesh filename=package://assets/l_tibia.stl
- link urdf_l_upper_arm_assembly: geometry collision mesh filename=package://assets/l_upper_arm.stl; visual mesh filename=package://assets/l_upper_arm.stl
- link urdf_l_upper_femur_assembly: geometry collision mesh filename=package://assets/l_upper_femur.stl; visual mesh filename=package://assets/l_upper_femur.stl
- link urdf_l_upper_forearm_assembly: geometry collision mesh filename=package://assets/l_upper_forearm.stl; visual mesh filename=package://assets/l_upper_forearm.stl
- link urdf_l_wrist_assembly: geometry collision mesh filename=package://assets/l_hand.stl; collision mesh filename=package://assets/l_wrist.stl
- link urdf_lower_femur_assembly: geometry collision mesh filename=package://assets/lower_femur.stl; visual mesh filename=package://assets/lower_femur.stl
- link urdf_lower_femur_assembly_2: geometry collision mesh filename=package://assets/lower_femur.stl; visual mesh filename=package://assets/lower_femur.stl
- link urdf_r_elbow_assembly: geometry collision mesh filename=package://assets/r_elbow.stl; visual mesh filename=package://assets/r_elbow.stl
- link urdf_r_lower_forearm_assembly: geometry collision mesh filename=package://assets/r_lower_forearm.stl; visual mesh filename=package://assets/r_lower_forearm.stl
- link urdf_r_shoulder_assembly: geometry collision mesh filename=package://assets/r_shoulder.stl; visual mesh filename=package://assets/r_shoulder.stl
- link urdf_r_tibia_assembly: geometry collision mesh filename=package://assets/foot.stl; collision mesh filename=package://assets/r_tibia.stl
- link urdf_r_upper_arm_assembly: geometry collision mesh filename=package://assets/r_upper_arm.stl; visual mesh filename=package://assets/r_upper_arm.stl
- link urdf_r_upper_femur_assemby: geometry collision mesh filename=package://assets/r_upper_femur.stl; visual mesh filename=package://assets/r_upper_femur.stl
- link urdf_r_upper_forearm_assembly: geometry collision mesh filename=package://assets/r_upper_forearm.stl; visual mesh filename=package://assets/r_upper_forearm.stl
- link urdf_r_wrist_assembly: geometry collision mesh filename=package://assets/r_hand.stl; collision mesh filename=package://assets/r_wrist.stl
- link urdf_simplified_torso_sub_assembly: geometry collision mesh filename=package://assets/head.stl; collision mesh filename=package://assets/simplified_torso.stl
