Commit message: limits correctionm

File: robot_gazebo.urdf (robot description, URDF)
Before this commit: robot robot_v1, 24 links, 23 joints
Joints:
- joint left_ankle_pitch_joint: limit lower=-0.785398 upper=0.785398 effort=10 velocity=10 -> lower=-0.785398 upper=0.785398 effort=100 velocity=100
- joint left_elbow_pitch_joint_X6: limit lower=-1.5708 upper=1.5708 effort=10 velocity=10 -> lower=-1.5708 upper=1.5708 effort=100 velocity=100
- joint left_hip_pitch_joint: limit lower=-2.53073 upper=1.5708 effort=10 velocity=10 -> lower=-2.53073 upper=1.5708 effort=100 velocity=100
- joint left_hip_roll_joint: limit lower=-0.349066 upper=3.14159 effort=10 velocity=10 -> lower=-0.349066 upper=3.14159 effort=100 velocity=100
- joint left_hip_yaw_joint: limit lower=-1.5708 upper=1.5708 effort=10 velocity=10 -> lower=-1.5708 upper=1.5708 effort=100 velocity=100
- joint left_knee_joint: limit lower=-1.5708 upper=-0 effort=10 velocity=10 -> lower=0.191906 upper=-2.33882 effort=100 velocity=100
- joint left_shoulder_pitch_joint_X6: limit lower=-3.14159 upper=1.5708 effort=10 velocity=10 -> lower=-3.14159 upper=1.5708 effort=100 velocity=100
- joint left_shoulder_roll_joint_X6: limit lower=-1.74533 upper=1.39626 effort=10 velocity=10 -> lower=-0.1 upper=3.0 effort=100 velocity=100
- joint left_shoulder_yaw_joint_X4: limit lower=-2.35619 upper=2.35619 effort=10 velocity=10 -> lower=-2.35619 upper=2.35619 effort=100 velocity=100
- joint left_wrist_roll_joint_X4: limit lower=-1.39626 upper=1.74533 effort=10 velocity=10 -> lower=-1.39626 upper=1.74533 effort=100 velocity=100
- joint left_wrist_yaw_joint_X4: limit lower=-2.35619 upper=2.35619 effort=10 velocity=10 -> lower=-2.35619 upper=2.35619 effort=100 velocity=100
- joint right_ankle_pitch_joint: limit lower=-0.785398 upper=0.785398 effort=10 velocity=10 -> lower=-0.785398 upper=0.785398 effort=100 velocity=100
- joint right_elbow_pitch_joint_X6: limit lower=-1.5708 upper=1.5708 effort=10 velocity=10 -> lower=-1.5708 upper=1.5708 effort=100 velocity=100
- joint right_hip_pitch_joint: limit lower=-2.51486 upper=1.58667 effort=10 velocity=10 -> lower=-2.51486 upper=1.58667 effort=100 velocity=100
- joint right_hip_roll_joint: limit lower=-3.14005 upper=0.35061 effort=10 velocity=10 -> lower=-3.14005 upper=0.35061 effort=100 velocity=100
- joint right_hip_yaw_joint: limit lower=-1.57082 upper=1.57077 effort=10 velocity=10 -> lower=-1.57082 upper=1.57077 effort=100 velocity=100
- joint right_knee_joint: limit lower=-0.191906 upper=2.33882 effort=10 velocity=10 -> lower=-0.191906 upper=2.33882 effort=100 velocity=100
- joint right_shoulder_pitch_joint_X6: limit lower=-3.14159 upper=1.5708 effort=10 velocity=10 -> lower=-3.14159 upper=1.5708 effort=100 velocity=100
- joint right_shoulder_roll_joint_X6: limit lower=-1.39626 upper=1.74533 effort=10 velocity=10 -> lower=-3.0 upper=0.1 effort=100 velocity=100
- joint right_shoulder_yaw_joint_X4: limit lower=-2.35619 upper=2.35619 effort=10 velocity=10 -> lower=-2.35619 upper=2.35619 effort=100 velocity=100
- joint right_wrist_roll_joint_X4: limit lower=-1.74533 upper=1.39626 effort=10 velocity=10 -> lower=-1.74533 upper=1.39626 effort=100 velocity=100
- joint right_wrist_yaw_joint_X4: limit lower=-2.35619 upper=2.35619 effort=10 velocity=10 -> lower=-2.35619 upper=2.35619 effort=100 velocity=100
- joint waist_yaw_joint: limit lower=-1.5708 upper=1.5708 effort=10 velocity=10 -> lower=-1.5708 upper=1.5708 effort=100 velocity=100

Commit message: update URDF pipeline: strip hand meshes, fix xacro output formatting
- urdf_simplify.py: add l_hand/r_hand to stripped mesh patterns
- split_urdf.py: sort joints by kinematic chain order (proximal→distal),
  add fixed_legs xacro property with comment block, remove space before />
- build_description.py: no changes (--fixed-legs flag already supported)
- urdf_simplify.md: restructure docs with build_description quick start,
  add step 4 (split_urdf.py) documentation

File: robot_gazebo.urdf (robot description, URDF)
Before this commit: robot robot_v1, 24 links, 23 joints
Links:
- link urdf_l_wrist_assembly: geometry collision mesh filename=package://meshes/collision/l_wrist.stl; visual mesh filename=package://meshes/visual/l_wrist.stl
- link urdf_r_wrist_assembly: geometry collision mesh filename=package://meshes/collision/r_wrist.stl; visual mesh filename=package://meshes/visual/r_wrist.stl

File: robot_simplified.urdf (robot description, URDF)
Before this commit: robot robot_v1, 24 links, 23 joints
Links:
- link urdf_l_wrist_assembly: geometry collision mesh filename=package://assets/l_wrist.stl; visual mesh filename=package://assets/l_wrist.stl
- link urdf_r_wrist_assembly: geometry collision mesh filename=package://assets/r_wrist.stl; visual mesh filename=package://assets/r_wrist.stl

File: robot_with_limits.urdf (robot description, URDF)
Before this commit: robot robot_v1, 24 links, 23 joints
Links:
- link urdf_l_wrist_assembly: geometry collision mesh filename=package://assets/l_wrist.stl; visual mesh filename=package://assets/l_wrist.stl
- link urdf_r_wrist_assembly: geometry collision mesh filename=package://assets/r_wrist.stl; visual mesh filename=package://assets/r_wrist.stl
